File: H1AR10/Design/H1AR10.sch (EAGLE design)
At the start: 42 parts, among them P1 HEXABIT_17.32_NO_P3, U1 STM32F091CBU6, U2 FT230XQ, U3 TI_NATIONAL_SEMICONDUCTOR_LM3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, X1 XTALL_CSTCE8M00G52, X3 USB-B-H

Commit message: final un-checked
Parts:
- removed JP1: (no value), Hexabitz:JP1E
- removed U3: TI_NATIONAL_SEMICONDUCTOR_LM3940IMP-3.3TI_NATIONAL_SEMICOND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, TI National Semiconductor - LM3940IMP-3.3:TI_NATIONAL_SEMICONDUCTOR_LM3940IMP-3.3TI_NATIONAL_SEMICONDUCTOR_LM3940IMP-3.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
- added PWR: 3-644456-2, Hexabitz:3-644456-2
- added U4: FT230XQ-R, Hexabitz:FT230XQ-R
- C16: device Hexabitz:C-EUC3225 -> Hexabitz:C-3225TDK_C3225X5R0J107M250AC_0_0
- D1, D2, D3: value VLMS1300-GS08 -> RED
- U2: value FT230XQ -> LM3940IMP-3.3; device Hexabitz:FT230XQ -> Hexabitz:LM3940IMP-3.3; OCTOPART_URL https://octopart.com/ft230xq-r-ftdi-22061504 -> (none)
Connections:
- removed net VDD2: C15.1, U2.!RESET, U2.3V3OUT
- net GND: now also U1.PC13, U2.GND_2, U4.GND@13, U4.GND@17, U4.GND@3; no longer U1.PB13, U1.PB7, U3.GND, U3.TAB
- net N$10: now also U4.CBUS1; no longer U2.CBUS1
- net N$11: now also U4.USBDM; no longer U2.USBDM
- net N$12: now also U4.USBDP; no longer U2.USBDP
- net N$15: now also PWR.1; no longer JP1.2
- net N$16: now also U2.IN; no longer U3.IN
- net N$17: now also PWR.2; no longer JP1.1
- net N$3: now also U4.CBUS2; no longer U2.CBUS2
- net UART1_CTS: now also U4.!CTS!; no longer U2.!CTS
- net UART1_RTS: now also U4.!RTS!; no longer U2.!RTS
- net UART1_RX: now also U4.TXD; no longer U2.TXD
- net UART1_TX: now also U4.RXD; no longer U2.RXD
- net VBUS_SENSE: now also U4.CBUS3; no longer U2.CBUS3
- net VDD: now also C15.1, U2.OUT, U4.!RESET!, U4.3V3OUT, U4.VCC, U4.VCCIO; no longer U2.VCC, U2.VCCIO, U3.OUT
Other:
- moved on the sheet: C10, C11, C12, C13, C14, C15, C17, D2, D3, FB2, R4, R5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

Commit message: rotate "C" & "D" pads 90 degrees chage X2 (label) to PUSB* change the led pin to (PB1) pin make "R" pad away enough form "B" pad fix some clearnce  issues
Parts:
- removed D1: RED, Hexabitz:VLMS1300-GS08
- removed U4: FT230XQ-R, Hexabitz:FT230XQ-R
- removed X3: USB-B-H, Hexabitz:USB-B-H
- added D4: RED, Hexabitz:VLMS1300-GS08
- added PUSB*: USB-B, Hexabitz:PN61729-S
- added U3: LM3940IMP-3.3, Hexabitz:LM3940IMP-3.3
- D3: value RED -> Green
- U2: value LM3940IMP-3.3 -> FT230XQ-R; device Hexabitz:LM3940IMP-3.3 -> Hexabitz:FT230XQ-R
Connections:
- removed net N$1: R1.2, U1.PA15
- removed net N$4: D1.A, R1.1
- new net N$18: D4.A, R1.1
- new net N$19: R1.2, U1.PB1
- net GND: now also D4.C, PUSB*.4, PUSB*.S1, PUSB*.S2, U2.GND@13, U2.GND@17, U2.GND@3, U3.GND, U3.GND_2; no longer D1.C, U2.GND, U2.GND_2, U4.GND@13, U4.GND@17, U4.GND@3, X3.GND
- net N$10: now also U2.CBUS1; no longer U4.CBUS1
- net N$11: now also U2.USBDM; no longer U4.USBDM
- net N$12: now also U2.USBDP; no longer U4.USBDP
- net N$13: now also PUSB*.3; no longer X3.D+
- net N$14: now also PUSB*.2; no longer X3.D-
- net N$16: now also U3.IN; no longer U2.IN
- net N$17: now also PUSB*.1; no longer X3.VBUS
- net N$3: now also U2.CBUS2; no longer U4.CBUS2
- net UART1_CTS: now also U2.!CTS!; no longer U4.!CTS!
- net UART1_RTS: now also U2.!RTS!; no longer U4.!RTS!
- net UART1_RX: now also U2.TXD; no longer U4.TXD
- net UART1_TX: now also U2.RXD; no longer U4.RXD
- net VBUS_SENSE: now also U2.CBUS3; no longer U4.CBUS3
- net VDD: now also U2.!RESET!, U2.3V3OUT, U2.VCC, U2.VCCIO, U3.OUT; no longer U2.OUT, U4.!RESET!, U4.3V3OUT, U4.VCC, U4.VCCIO
Other:
- moved on the sheet: C16, R1

Commit message: no message
Parts:
- renumbered D4 to D1
Changed lines of the file:
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@@
 <setting verticaltext="up"/>
 </settings>
-<grid distance="50" unitdist="mil" unit="mm" style="lines" multiple="1" display="yes" altdistance="0.01" altunitdist="inch" altunit="inch"/>
+<grid distance="0.1" unitdist="inch" unit="inch" style="lines" multiple="1" display="no" altdistance="0.01" altunitdist="inch" altunit="inch"/>
 <layers>
 <layer number="1" name="Top" color="4" fill="1" visible="no" active="no"/>
@@
 <attribute name="TOLERANCE" value="5%"/>
 </part>
-<part name="D4" library="Hexabitz" deviceset="VLMS1300-GS08" device="" value="RED">
+<part name="D1" library="Hexabitz" deviceset="VLMS1300-GS08" device="" value="RED">
 <attribute name="MFN" value="Vishay"/>
 <attribute name="MPN" value="VLMS1300-GS08"/>
@@
 <attribute name="VALUE" x="231.14" y="178.562" size="1.778" layer="96" rot="R180"/>
 </instance>
-<instance part="D4" gate="G$1" x="237.49" y="175.26" smashed="yes" rot="MR0">
-<attribute name="NAME" x="242.062" y="171.704" size="1.778" layer="95" rot="MR0"/>
-<attribute name="VALUE" x="242.062" y="179.705" size="1.778" layer="96" rot="MR0"/>
+<instance part="D1" gate="G$1" x="237.49" y="175.26" smashed="yes" rot="MR0">
+<attribute name="NAME" x="240.792" y="179.324" size="1.778" layer="95" rot="MR0"/>
+<attribute name="VALUE" x="242.062" y="170.815" size="1.778" layer="96" rot="MR0"/>
 </instance>
 <instance part="GND22" gate="1" x="245.11" y="167.64" smashed="yes">
@@
 <pinref part="GND22" gate="1" pin="GND"/>
 <wire x1="245.11" y1="170.18" x2="245.11" y2="175.26" width="0.1524" layer="91"/>
-<pinref part="D4" gate="G$1" pin="C"/>
+<pinref part="D1" gate="G$1" pin="C"/>
 <wire x1="245.11" y1="175.26" x2="242.57" y2="175.26" width="0.1524" layer="91"/>
 </segment>
@@
 <segment>
 <pinref part="R1" gate="G$1" pin="1"/>
-<pinref part="D4" gate="G$1" pin="A"/>
+<pinref part="D1" gate="G$1" pin="A"/>
 <wire x1="232.41" y1="175.26" x2="234.95" y2="175.26" width="0.1524" layer="91"/>
 </segment>

Commit message: no message
Parts:
- D2: value RED -> YELLOW; MPN VLMS1300-GS08 -> VLMY1300-GS08; OCTOPART_URL https://octopart.com/vlms1300-gs08-vishay-21709201 -> https://octopart.com/vlmy1300-gs08-vishay-21709204?r=sp
- D3: value Green -> ORANGE; MPN VLMTG1300-GS08 -> VLMO1300-GS08; OCTOPART_URL https://octopart.com/vlmtg1300-gs08-vishay-21709202 -> https://octopart.com/vlmo1300-gs08-vishay-21709200?r=sp#
Other:
- moved on the sheet: D2, D3, R6, R7
Changed lines of the file:
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@@
 <setting verticaltext="up"/>
 </settings>
-<grid distance="0.1" unitdist="inch" unit="inch" style="lines" multiple="1" display="no" altdistance="0.01" altunitdist="inch" altunit="inch"/>
+<grid distance="0.1" unitdist="inch" unit="mil" style="lines" multiple="1" display="no" altdistance="0.01" altunitdist="inch" altunit="inch"/>
 <layers>
 <layer number="1" name="Top" color="4" fill="1" visible="no" active="no"/>
@@
 <attribute name="VOLTAGE_RATING" value="50"/>
 </part>
-<part name="D3" library="Hexabitz" deviceset="VLMS1300-GS08" device="" value="Green">
+<part name="D3" library="Hexabitz" deviceset="VLMS1300-GS08" device="" value="ORANGE">
 <attribute name="MFN" value="Vishay"/>
-<attribute name="MPN" value="VLMTG1300-GS08 "/>
-<attribute name="OCTOPART_URL" value="https://octopart.com/vlmtg1300-gs08-vishay-21709202"/>
+<attribute name="MPN" value="VLMO1300-GS08
+"/>
+<attribute name="OCTOPART_URL" value="https://octopart.com/vlmo1300-gs08-vishay-21709200?r=sp#"/>
 </part>
-<part name="D2" library="Hexabitz" deviceset="VLMS1300-GS08" device="" value="RED">
+<part name="D2" library="Hexabitz" deviceset="VLMS1300-GS08" device="" value="YELLOW">
 <attribute name="MFN" value="Vishay"/>
-<attribute name="MPN" value="VLMS1300-GS08"/>
-<attribute name="OCTOPART_URL" value="https://octopart.com/vlms1300-gs08-vishay-21709201"/>
+<attribute name="MPN" value="VLMY1300-GS08"/>
+<attribute name="OCTOPART_URL" value="https://octopart.com/vlmy1300-gs08-vishay-21709204?r=sp"/>
 </part>
 <part name="FB2" library="Hexabitz" deviceset="FB-TDK_MMZ1608Y300B" device="" value="FB-TDK_MMZ1608Y300B">
@@
 </plain>
 <instances>
-<instance part="R7" gate="G$1" x="227.33" y="76.2" smashed="yes" rot="R90">
-<attribute name="NAME" x="228.6" y="78.9686" size="1.778" layer="95"/>
-<attribute name="VALUE" x="236.22" y="74.422" size="1.778" layer="96" rot="R180"/>
-</instance>
-<instance part="R6" gate="G$1" x="240.03" y="76.2" smashed="yes" rot="R90">
-<attribute name="NAME" x="241.3" y="78.9686" size="1.778" layer="95"/>
-<attribute name="VALUE" x="241.3" y="72.898" size="1.778" layer="96"/>
+<instance part="R7" gate="G$1" x="224.79" y="76.2" smashed="yes" rot="R90">
+<attribute name="NAME" x="226.06" y="78.9686" size="1.778" layer="95"/>
+<attribute name="VALUE" x="233.68" y="74.422" size="1.778" layer="96" rot="R180"/>
+</instance>
+<instance part="R6" gate="G$1" x="242.57" y="76.2" smashed="yes" rot="R90">
+<attribute name="NAME" x="243.84" y="78.9686" size="1.778" layer="95"/>
+<attribute name="VALUE" x="243.84" y="72.898" size="1.778" layer="96"/>
 </instance>
 <instance part="SUPPLY14" gate="G$1" x="233.68" y="44.45" smashed="yes" rot="R180">
@@
 <attribute name="VALUE" x="118.364" y="84.201" size="1.778" layer="96"/>
 </instance>
-<instance part="D3" gate="G$1" x="240.03" y="63.5" smashed="yes" rot="MR270">
-<attribute name="NAME" x="243.078" y="68.326" size="1.778" layer="95" rot="MR180"/>
-<attribute name="VALUE" x="243.078" y="64.135" size="1.778" layer="96" rot="MR180"/>
-</instance>
-<instance part="D2" gate="G$1" x="227.33" y="63.5" smashed="yes" rot="MR270">
-<attribute name="NAME" x="229.108" y="68.326" size="1.778" layer="95" rot="MR180"/>
-<attribute name="VALUE" x="229.108" y="64.135" size="1.778" layer="96" rot="MR180"/>
+<instance part="D3" gate="G$1" x="242.57" y="63.5" smashed="yes" rot="MR270">
+<attribute name="NAME" x="245.618" y="68.326" size="1.778" layer="95" rot="MR180"/>
+<attribute name="VALUE" x="245.618" y="64.135" size="1.778" layer="96" rot="MR180"/>
+</instance>
+<instance part="D2" gate="G$1" x="224.79" y="63.5" smashed="yes" rot="MR270">
+<attribute name="NAME" x="226.568" y="68.326" size="1.778" layer="95" rot="MR180"/>
+<attribute name="VALUE" x="226.568" y="64.135" size="1.778" layer="96" rot="MR180"/>
 </instance>
 <instance part="FB2" gate="G$1" x="72.39" y="154.94" smashed="yes" rot="R180">
@@
 <segment>
 <pinref part="R7" gate="G$1" pin="2"/>
-<wire x1="227.33" y1="87.63" x2="227.33" y2="81.28" width="0.1524" layer="91"/>
-<wire x1="200.66" y1="87.63" x2="227.33" y2="87.63" width="0.1524" layer="91"/>
+<wire x1="224.79" y1="87.63" x2="224.79" y2="81.28" width="0.1524" layer="91"/>
+<wire x1="200.66" y1="87.63" x2="224.79" y2="87.63" width="0.1524" layer="91"/>
 <pinref part="U2" gate="G$1" pin="CBUS2"/>
 </segment>
@@
 <segment>
 <pinref part="R6" gate="G$1" pin="2"/>
-<wire x1="240.03" y1="81.28" x2="240.03" y2="90.17" width="0.1524" layer="91"/>
-<wire x1="240.03" y1="90.17" x2="200.66" y2="90.17" width="0.1524" layer="91"/>
+<wire x1="242.57" y1="81.28" x2="242.57" y2="90.17" width="0.1524" layer="91"/>
+<wire x1="242.57" y1="90.17" x2="200.66" y2="90.17" width="0.1524" layer="91"/>
 <pinref part="U2" gate="G$1" pin="CBUS1"/>
 </segment>
@@
 <segment>
 <pinref part="R6" gate="G$1" pin="1"/>
-<wire x1="240.03" y1="71.12" x2="240.03" y2="68.58" width="0.1524" layer="91"/>
+<wire x1="242.57" y1="71.12" x2="242.57" y2="68.58" width="0.1524" layer="91"/>
 <pinref part="D3" gate="G$1" pin="C"/>
 </segment>
@@
 <segment>
 <pinref part="R7" gate="G$1" pin="1"/>
-<wire x1="227.33" y1="68.58" x2="227.33" y2="71.12" width="0.1524" layer="91"/>
+<wire x1="224.79" y1="68.58" x2="224.79" y2="71.12" width="0.1524" layer="91"/>
 <pinref part="D2" gate="G$1" pin="C"/>
 </segment>
@@
 <net name="VDD" class="0">
 <segment>
-<wire x1="227.33" y1="60.96" x2="227.33" y2="50.8" width="0.1524" layer="91"/>
-<wire x1="227.33" y1="50.8" x2="233.68" y2="50.8" width="0.1524" layer="91"/>
-<wire x1="233.68" y1="50.8" x2="240.03" y2="50.8" width="0.1524" layer="91"/>
-<wire x1="240.03" y1="50.8" x2="240.03" y2="60.96" width="0.1524" layer="91"/>
+<wire x1="224.79" y1="60.96" x2="224.79" y2="50.8" width="0.1524" layer="91"/>
+<wire x1="224.79" y1="50.8" x2="233.68" y2="50.8" width="0.1524" layer="91"/>
+<wire x1="233.68" y1="50.8" x2="242.57" y2="50.8" width="0.1524" layer="91"/>
+<wire x1="242.57" y1="50.8" x2="242.57" y2="60.96" width="0.1524" layer="91"/>
 <pinref part="SUPPLY14" gate="G$1" pin="VDD"/>
 <wire x1="233.68" y1="46.99" x2="233.68" y2="50.8" width="0.1524" layer="91"/>
